File: ram.sch (KiCad schematic (older format))
At the start: 4 parts, among them U2 XX4256, U3 XX4256

Commit message: Switch out the MOS 6529
Parts:
- U2, U3: footprint MODULE -> Package_DIP:DIP-20_W7.62mm_Socket
Changed lines of the file:
@@
 F 0 "U3" H 8718 6436 50  0000 L CNN
 F 1 "XX4256" H 8718 6345 50  0000 L CNN
-F 2 "MODULE" H 8490 6390 50  0001 C CNN
+F 2 "Package_DIP:DIP-20_W7.62mm_Socket" H 8490 6390 50  0001 C CNN
 F 3 "DOCUMENTATION" H 8490 6390 50  0001 C CNN
 	1    8490 6390
@@
 F 0 "U2" H 2098 9946 50  0000 L CNN
 F 1 "XX4256" H 2098 9855 50  0000 L CNN
-F 2 "MODULE" H 1870 9900 50  0001 C CNN
+F 2 "Package_DIP:DIP-20_W7.62mm_Socket" H 1870 9900 50  0001 C CNN
 F 3 "DOCUMENTATION" H 1870 9900 50  0001 C CNN
 	2    1870 9900
@@
 F 0 "U2" H 8490 5405 50  0000 C CNN
 F 1 "XX4256" H 8490 5314 50  0000 C CNN
-F 2 "MODULE" H 8490 4690 50  0001 C CNN
+F 2 "Package_DIP:DIP-20_W7.62mm_Socket" H 8490 4690 50  0001 C CNN
 F 3 "DOCUMENTATION" H 8490 4690 50  0001 C CNN
 	1    8490 4690
@@
 F 0 "U3" H 4113 9946 50  0000 L CNN
 F 1 "XX4256" H 4113 9855 50  0000 L CNN
-F 2 "MODULE" H 3885 9900 50  0001 C CNN
+F 2 "Package_DIP:DIP-20_W7.62mm_Socket" H 3885 9900 50  0001 C CNN
 F 3 "DOCUMENTATION" H 3885 9900 50  0001 C CNN
 	2    3885 9900

Commit message: Start working on PCB
Parts:
- C3: renamed from C1; footprint (none) -> Capacitor_SMD:C_0805_2012Metric_Pad1.18x1.45mm_HandSolder
- C4: renamed from C2; footprint (none) -> Capacitor_SMD:C_0805_2012Metric_Pad1.18x1.45mm_HandSolder
- renumbered U2 to U4, U3 to U5
Changed lines of the file:
@@
 P 8490 6390
 AR Path="/63A919D8" Ref="U?"  Part="2"
-AR Path="/62E48B71/63A919D8" Ref="U3"  Part="1"
-F 0 "U3" H 8718 6436 50  0000 L CNN
-F 1 "XX4256" H 8718 6345 50  0000 L CNN
+AR Path="/62E48B71/63A919D8" Ref="U5"  Part="1"
+F 0 "U5" H 8490 7105 50  0000 C CNN
+F 1 "XX4256" H 8490 7014 50  0000 C CNN
 F 2 "Package_DIP:DIP-20_W7.62mm_Socket" H 8490 6390 50  0001 C CNN
 F 3 "DOCUMENTATION" H 8490 6390 50  0001 C CNN
@@
 P 1870 9900
 AR Path="/63A91A52" Ref="U?"  Part="1"
-AR Path="/62E48B71/63A91A52" Ref="U2"  Part="2"
-F 0 "U2" H 2098 9946 50  0000 L CNN
+AR Path="/62E48B71/63A91A52" Ref="U4"  Part="2"
+F 0 "U4" H 2098 9946 50  0000 L CNN
 F 1 "XX4256" H 2098 9855 50  0000 L CNN
 F 2 "Package_DIP:DIP-20_W7.62mm_Socket" H 1870 9900 50  0001 C CNN
@@
 P 8490 4690
 AR Path="/63A91A85" Ref="U?"  Part="1"
-AR Path="/62E48B71/63A91A85" Ref="U2"  Part="1"
-F 0 "U2" H 8490 5405 50  0000 C CNN
+AR Path="/62E48B71/63A91A85" Ref="U4"  Part="1"
+F 0 "U4" H 8490 5405 50  0000 C CNN
 F 1 "XX4256" H 8490 5314 50  0000 C CNN
 F 2 "Package_DIP:DIP-20_W7.62mm_Socket" H 8490 4690 50  0001 C CNN
@@
 P 1335 9895
 AR Path="/63ABB0AA" Ref="C?"  Part="1"
-AR Path="/62E48B71/63ABB0AA" Ref="C1"  Part="1"
+AR Path="/62E48B71/63ABB0AA" Ref="C3"  Part="1"
 AR Path="/63A22C28/63ABB0AA" Ref="C?"  Part="1"
-F 0 "C1" H 1220 9941 50  0000 R CNN
+F 0 "C3" H 1220 9941 50  0000 R CNN
 F 1 "100n" H 1220 9850 50  0000 R CNN
-F 2 "" H 1373 9745 50  0001 C CNN
+F 2 "Capacitor_SMD:C_0805_2012Metric_Pad1.18x1.45mm_HandSolder" H 1373 9745 50  0001 C CNN
 F 3 "~" H 1335 9895 50  0001 C CNN
 	1    1335 9895
@@
 P 3350 9895
 AR Path="/63AC07CB" Ref="C?"  Part="1"
-AR Path="/62E48B71/63AC07CB" Ref="C2"  Part="1"
+AR Path="/62E48B71/63AC07CB" Ref="C4"  Part="1"
 AR Path="/63A22C28/63AC07CB" Ref="C?"  Part="1"
-F 0 "C2" H 3235 9941 50  0000 R CNN
+F 0 "C4" H 3235 9941 50  0000 R CNN
 F 1 "100n" H 3235 9850 50  0000 R CNN
-F 2 "" H 3388 9745 50  0001 C CNN
+F 2 "Capacitor_SMD:C_0805_2012Metric_Pad1.18x1.45mm_HandSolder" H 3388 9745 50  0001 C CNN
 F 3 "~" H 3350 9895 50  0001 C CNN
 	1    3350 9895
@@
 P 3885 9900
 AR Path="/63AC49C2" Ref="U?"  Part="2"
-AR Path="/62E48B71/63AC49C2" Ref="U3"  Part="2"
-F 0 "U3" H 4113 9946 50  0000 L CNN
+AR Path="/62E48B71/63AC49C2" Ref="U5"  Part="2"
+F 0 "U5" H 4113 9946 50  0000 L CNN
 F 1 "XX4256" H 4113 9855 50  0000 L CNN
 F 2 "Package_DIP:DIP-20_W7.62mm_Socket" H 3885 9900 50  0001 C CNN
