File: ras_cas_gen.sch (KiCad schematic (older format))
At the start: 10 parts, among them U12 74HCT74, U13 74HCT74, U4 74LS257, U5 74LS257, U6 GAL20V8

Commit message: Start working on PCB
Parts:
- C1: renamed from C9; footprint (none) -> Capacitor_SMD:C_0805_2012Metric_Pad1.18x1.45mm_HandSolder
- C5: renamed from C11; footprint (none) -> Capacitor_SMD:C_0805_2012Metric_Pad1.18x1.45mm_HandSolder
- C6: renamed from C12; footprint (none) -> Capacitor_SMD:C_0805_2012Metric_Pad1.18x1.45mm_HandSolder
- U6: footprint MODULE -> Package_DIP:DIP-24_W7.62mm_Socket
- U7: renamed from U12; footprint (none) -> Package_SO:SOIC-14_3.9x8.7mm_P1.27mm
- U8: renamed from U13; footprint (none) -> Package_SO:SOIC-14_3.9x8.7mm_P1.27mm
- renumbered C4 to C2, C3 to C7, U4 to U2, U5 to U3
Changed lines of the file:
@@
 AR Path="/63A64678" Ref="C?"  Part="1"
 AR Path="/62E48B71/63A64678" Ref="C?"  Part="1"
-AR Path="/63A22C28/63A64678" Ref="C3"  Part="1"
-F 0 "C3" H 4530 3256 50  0000 L CNN
+AR Path="/63A22C28/63A64678" Ref="C7"  Part="1"
+F 0 "C7" H 4530 3256 50  0000 L CNN
 F 1 "100n" H 4530 3165 50  0000 L CNN
 F 2 "Capacitor_SMD:C_0805_2012Metric_Pad1.18x1.45mm_HandSolder" H 4453 3060 50  0001 C CNN
@@
 AR Path="/63A64692" Ref="U?"  Part="1"
 AR Path="/62E48B71/63A64692" Ref="U?"  Part="1"
-AR Path="/63A22C28/63A64692" Ref="U5"  Part="1"
-F 0 "U5" H 10785 4900 50  0000 C CNN
+AR Path="/63A22C28/63A64692" Ref="U3"  Part="1"
+F 0 "U3" H 10785 4900 50  0000 C CNN
 F 1 "74LS257" H 10785 4600 50  0000 C CNN
 F 2 "Package_SO:SOIC-16_3.9x9.9mm_P1.27mm" H 10735 4750 50  0001 C CNN
@@
 AR Path="/63A64698" Ref="U?"  Part="1"
 AR Path="/62E48B71/63A64698" Ref="U?"  Part="1"
-AR Path="/63A22C28/63A64698" Ref="U4"  Part="1"
-F 0 "U4" H 10785 3200 50  0000 C CNN
+AR Path="/63A22C28/63A64698" Ref="U2"  Part="1"
+F 0 "U2" H 10785 3200 50  0000 C CNN
 F 1 "74LS257" H 10785 2900 50  0000 C CNN
 F 2 "Package_SO:SOIC-16_3.9x9.9mm_P1.27mm" H 10735 3050 50  0001 C CNN
@@
 AR Path="/63A6467E" Ref="C?"  Part="1"
 AR Path="/62E48B71/63A6467E" Ref="C?"  Part="1"
-AR Path="/63A22C28/63A6467E" Ref="C4"  Part="1"
-F 0 "C4" H 12600 4701 50  0000 L CNN
+AR Path="/63A22C28/63A6467E" Ref="C2"  Part="1"
+F 0 "C2" H 12600 4701 50  0000 L CNN
 F 1 "100n" H 12600 4610 50  0000 L CNN
 F 2 "Capacitor_SMD:C_0805_2012Metric_Pad1.18x1.45mm_HandSolder" H 12523 4505 50  0001 C CNN
@@
 AR Path="/63A64654" Ref="C?"  Part="1"
 AR Path="/62E48B71/63A64654" Ref="C?"  Part="1"
-AR Path="/63A22C28/63A64654" Ref="C9"  Part="1"
-F 0 "C9" H 12600 3066 50  0000 L CNN
+AR Path="/63A22C28/63A64654" Ref="C1"  Part="1"
+F 0 "C1" H 12600 3066 50  0000 L CNN
 F 1 "100n" H 12600 2975 50  0000 L CNN
-F 2 "" H 12523 2870 50  0001 C CNN
+F 2 "Capacitor_SMD:C_0805_2012Metric_Pad1.18x1.45mm_HandSolder" H 12523 2870 50  0001 C CNN
 F 3 "~" H 12485 3020 50  0001 C CNN
 	1    12485 3020
@@
 $EndComp
 $Comp
-L 74xx:74LS74 U13
+L 74xx:74LS74 U8
 U 2 1 63CBD2CF
 P 6815 7340
-F 0 "U13" H 6945 7595 50  0000 C CNN
+F 0 "U8" H 6945 7595 50  0000 C CNN
 F 1 "74HCT74" H 6815 7730 50  0001 C CNN
-F 2 "" H 6815 7340 50  0001 C CNN
+F 2 "Package_SO:SOIC-14_3.9x8.7mm_P1.27mm" H 6815 7340 50  0001 C CNN
 F 3 "74xx/74hc_hct74.pdf" H 6815 7340 50  0001 C CNN
 	2    6815 7340
@@
 $EndComp
 $Comp
-L 74xx:74LS74 U12
+L 74xx:74LS74 U7
 U 3 1 63CBF300
 P 1540 10005
-F 0 "U12" H 1770 10051 50  0000 L CNN
+F 0 "U7" H 1770 10051 50  0000 L CNN
 F 1 "74HCT74" H 1770 9960 50  0000 L CNN
-F 2 "" H 1540 10005 50  0001 C CNN
+F 2 "Package_SO:SOIC-14_3.9x8.7mm_P1.27mm" H 1540 10005 50  0001 C CNN
 F 3 "74xx/74hc_hct74.pdf" H 1540 10005 50  0001 C CNN
 	3    1540 10005
@@
 $EndComp
 $Comp
-L 74xx:74LS74 U13
+L 74xx:74LS74 U8
 U 3 1 63CC059A
 P 3105 10005
-F 0 "U13" H 3335 10051 50  0000 L CNN
+F 0 "U8" H 3335 10051 50  0000 L CNN
 F 1 "74HCT74" H 3335 9960 50  0000 L CNN
-F 2 "" H 3105 10005 50  0001 C CNN
+F 2 "Package_SO:SOIC-14_3.9x8.7mm_P1.27mm" H 3105 10005 50  0001 C CNN
 F 3 "74xx/74hc_hct74.pdf" H 3105 10005 50  0001 C CNN
 	3    3105 10005
@@
 	5420 6080 5520 5980
 $Comp
-L 74xx:74LS74 U13
+L 74xx:74LS74 U8
 U 1 1 63CBBBB2
 P 6285 6795
-F 0 "U13" H 6430 7055 50  0000 C CNN
+F 0 "U8" H 6430 7055 50  0000 C CNN
 F 1 "74HCT74" H 6495 6515 50  0000 C CNN
-F 2 "" H 6285 6795 50  0001 C CNN
+F 2 "Package_SO:SOIC-14_3.9x8.7mm_P1.27mm" H 6285 6795 50  0001 C CNN
 F 3 "74xx/74hc_hct74.pdf" H 6285 6795 50  0001 C CNN
 	1    6285 6795
@@
 	5910 7340 6515 7340
 $Comp
-L 74xx:74LS74 U12
+L 74xx:74LS74 U7
 U 2 1 63D2ED5A
 P 6815 6080
-F 0 "U12" H 6945 6335 50  0000 C CNN
+F 0 "U7" H 6945 6335 50  0000 C CNN
 F 1 "74HCT74" H 6815 6470 50  0001 C CNN
-F 2 "" H 6815 6080 50  0001 C CNN
+F 2 "Package_SO:SOIC-14_3.9x8.7mm_P1.27mm" H 6815 6080 50  0001 C CNN
 F 3 "74xx/74hc_hct74.pdf" H 6815 6080 50  0001 C CNN
 	2    6815 6080
@@
 $EndComp
 $Comp
-L 74xx:74LS74 U12
+L 74xx:74LS74 U7
 U 1 1 63D2F89C
 P 6285 5535
-F 0 "U12" H 6430 5795 50  0000 C CNN
+F 0 "U7" H 6430 5795 50  0000 C CNN
 F 1 "74HCT74" H 6495 5255 50  0000 C CNN
-F 2 "" H 6285 5535 50  0001 C CNN
+F 2 "Package_SO:SOIC-14_3.9x8.7mm_P1.27mm" H 6285 5535 50  0001 C CNN
 F 3 "74xx/74hc_hct74.pdf" H 6285 5535 50  0001 C CNN
 	1    6285 5535
@@
 AR Path="/63ECD15A" Ref="C?"  Part="1"
 AR Path="/62E48B71/63ECD15A" Ref="C?"  Part="1"
-AR Path="/63A22C28/63ECD15A" Ref="C11"  Part="1"
-F 0 "C11" H 915 10051 50  0000 R CNN
+AR Path="/63A22C28/63ECD15A" Ref="C5"  Part="1"
+F 0 "C5" H 915 10051 50  0000 R CNN
 F 1 "100n" H 915 9960 50  0000 R CNN
-F 2 "" H 1068 9855 50  0001 C CNN
+F 2 "Capacitor_SMD:C_0805_2012Metric_Pad1.18x1.45mm_HandSolder" H 1068 9855 50  0001 C CNN
 F 3 "~" H 1030 10005 50  0001 C CNN
 	1    1030 10005
@@
 AR Path="/63EDC36A" Ref="C?"  Part="1"
 AR Path="/62E48B71/63EDC36A" Ref="C?"  Part="1"
-AR Path="/63A22C28/63EDC36A" Ref="C12"  Part="1"
-F 0 "C12" H 2480 10051 50  0000 R CNN
+AR Path="/63A22C28/63EDC36A" Ref="C6"  Part="1"
+F 0 "C6" H 2480 10051 50  0000 R CNN
 F 1 "100n" H 2480 9960 50  0000 R CNN
-F 2 "" H 2633 9855 50  0001 C CNN
+F 2 "Capacitor_SMD:C_0805_2012Metric_Pad1.18x1.45mm_HandSolder" H 2633 9855 50  0001 C CNN
 F 3 "~" H 2595 10005 50  0001 C CNN
 	1    2595 10005
@@
 F 0 "U6" H 6355 4225 50  0000 C CNN
 F 1 "GAL20V8" H 6355 4134 50  0000 C CNN
-F 2 "MODULE" H 6355 3310 50  0001 C CNN
+F 2 "Package_DIP:DIP-24_W7.62mm_Socket" H 6355 3310 50  0001 C CNN
 F 3 "DOCUMENTATION" H 6355 3310 50  0001 C CNN
 	1    6355 3310

Commit message: Fix address pins
Connections:
- net a0: no longer U6.6 (I5)
- net a1: no longer U6.7 (I6)
- net a12: now also U6.6 (I5)
- net a13: now also U6.7 (I6)
- net a14: now also U6.8 (I7)
- net a15: now also U6.9 (I8)
- net a2: no longer U6.8 (I7)
- net a3: no longer U6.9 (I8)
- net p6: now reaches U6.14 (I11), U8.5 (Q)
- net p7: now reaches U6.15 (O0), U8.9 (Q)
- net p1: now reaches U6.13 (I_~OE), U7.9 (Q)
- net p0: now reaches U6.11 (I10), U7.5 (Q)
Changed lines of the file:
@@
 Sheet 3 3
 Title "C16/+4 256 kB RAM Expansion"
-Date "2022-07-30"
+Date "2022-08-16"
 Rev "1git"
 Comp "SukkoPera"
@@
 	5090 3160 5190 3260
 Text Label 5190 3460 0    50   ~ 0
-a2
+a14
 Wire Wire Line
 	5605 3460 5190 3460
 Text Label 5190 3360 0    50   ~ 0
-a1
+a13
 Wire Wire Line
 	5605 3360 5190 3360
 Text Label 5190 3260 0    50   ~ 0
-a0
+a12
 Wire Wire Line
 	5605 3260 5190 3260
 Text Label 5190 3560 0    50   ~ 0
-a3
+a15
 Wire Wire Line
 	5605 3560 5190 3560
@@
 Wire Bus Line
 	9285 2250 9285 4950
+Text Label 6605 5435 0    50   ~ 0
+p0
+Text Label 7120 5980 0    50   ~ 0
+p1
+Text Label 6605 6695 0    50   ~ 0
+p6
+Text Label 7120 7240 0    50   ~ 0
+p7
 $EndSCHEMATC
