File: ras_cas_gen.sch (KiCad schematic (older format))
At the start: 10 parts, among them U2 74LS257, U3 74LS257, U6 GAL20V8, U7 74HCT74, U8 74HCT74

Commit message: Routing in progress
Connections:
- net VCC is gone; now on net +5V: C2.1, C7.1, U2.16 (VCC), U3.16 (VCC)
Changed lines of the file:
@@
 Sheet 3 3
 Title "Hannes256: C16/+4 256 kB RAM Expansion"
-Date "2022-08-16"
+Date "2022-09-19"
 Rev "1git"
 Comp "SukkoPera"
@@
 $EndComp
 $Comp
-L power:VCC #PWR?
-U 1 1 63A64684
-P 4415 2960
-AR Path="/63A64684" Ref="#PWR?"  Part="1"
-AR Path="/62E48B71/63A64684" Ref="#PWR?"  Part="1"
-AR Path="/63A22C28/63A64684" Ref="#PWR017"  Part="1"
-F 0 "#PWR017" H 4415 2810 50  0001 C CNN
-F 1 "VCC" H 4430 3133 50  0000 C CNN
-F 2 "" H 4415 2960 50  0001 C CNN
-F 3 "" H 4415 2960 50  0001 C CNN
-	1    4415 2960
-	1    0    0    -1
-$EndComp
-$Comp
 L power:GND #PWR?
 U 1 1 63A6468A
@@
 	1    0    0    -1
 $EndComp
-$Comp
-L power:VCC #PWR?
-U 1 1 63A6466C
-P 12485 4405
-AR Path="/63A6466C" Ref="#PWR?"  Part="1"
-AR Path="/62E48B71/63A6466C" Ref="#PWR?"  Part="1"
-AR Path="/63A22C28/63A6466C" Ref="#PWR018"  Part="1"
-F 0 "#PWR018" H 12485 4255 50  0001 C CNN
-F 1 "VCC" H 12485 4555 50  0000 C CNN
-F 2 "" H 12485 4405 50  0001 C CNN
-F 3 "" H 12485 4405 50  0001 C CNN
-	1    12485 4405
-	1    0    0    -1
-$EndComp
 Wire Wire Line
 	12485 4505 12485 4405
@@
 Text Notes 5730 4270 0    50   ~ 0
 ALL THE GLUE LOGIC WAS REPLACED\nWITH A SINGLE OLD-SKOOLZ GAL!
+Text Label 6605 5435 0    50   ~ 0
+p0
+Text Label 7120 5980 0    50   ~ 0
+p1
+Text Label 6605 6695 0    50   ~ 0
+p6
+Text Label 7120 7240 0    50   ~ 0
+p7
+$Comp
+L power:+5V #PWR?
+U 1 1 633D8DCD
+P 4415 2960
+AR Path="/633D8DCD" Ref="#PWR?"  Part="1"
+AR Path="/62E48B71/633D8DCD" Ref="#PWR?"  Part="1"
+AR Path="/63A22C28/633D8DCD" Ref="#PWR0106"  Part="1"
+F 0 "#PWR0106" H 4415 2810 50  0001 C CNN
+F 1 "+5V" H 4430 3133 50  0000 C CNN
+F 2 "" H 4415 2960 50  0001 C CNN
+F 3 "" H 4415 2960 50  0001 C CNN
+	1    4415 2960
+	1    0    0    -1
+$EndComp
+$Comp
+L power:+5V #PWR?
+U 1 1 633D9554
+P 12485 4405
+AR Path="/633D9554" Ref="#PWR?"  Part="1"
+AR Path="/62E48B71/633D9554" Ref="#PWR?"  Part="1"
+AR Path="/63A22C28/633D9554" Ref="#PWR0107"  Part="1"
+F 0 "#PWR0107" H 12485 4255 50  0001 C CNN
+F 1 "+5V" H 12500 4578 50  0000 C CNN
+F 2 "" H 12485 4405 50  0001 C CNN
+F 3 "" H 12485 4405 50  0001 C CNN
+	1    12485 4405
+	1    0    0    -1
+$EndComp
+$Comp
+L power:+5V #PWR?
+U 1 1 633E34D2
+P 12485 3790
+AR Path="/633E34D2" Ref="#PWR?"  Part="1"
+AR Path="/62E48B71/633E34D2" Ref="#PWR?"  Part="1"
+AR Path="/63A22C28/633E34D2" Ref="#PWR0108"  Part="1"
+F 0 "#PWR0108" H 12485 3640 50  0001 C CNN
+F 1 "+5V" H 12500 3963 50  0000 C CNN
+F 2 "" H 12485 3790 50  0001 C CNN
+F 3 "" H 12485 3790 50  0001 C CNN
+	1    12485 3790
+	1    0    0    -1
+$EndComp
+$Comp
+L power:VCC #PWR0109
+U 1 1 633E54A0
+P 12855 3790
+F 0 "#PWR0109" H 12855 3640 50  0001 C CNN
+F 1 "VCC" H 12870 3963 50  0000 C CNN
+F 2 "" H 12855 3790 50  0001 C CNN
+F 3 "" H 12855 3790 50  0001 C CNN
+	1    12855 3790
+	1    0    0    -1
+$EndComp
+Wire Wire Line
+	12855 3790 12855 3890
+Wire Wire Line
+	12855 3890 12485 3890
+Wire Wire Line
+	12485 3890 12485 3790
 Wire Bus Line
 	5420 5535 5420 7340
@@
 Wire Bus Line
 	9285 2250 9285 4950
-Text Label 6605 5435 0    50   ~ 0
-p0
-Text Label 7120 5980 0    50   ~ 0
-p1
-Text Label 6605 6695 0    50   ~ 0
-p6
-Text Label 7120 7240 0    50   ~ 0
-p7
 $EndSCHEMATC

Commit message: Switch to 41256 RAM This will handle the refresh properly despite needing 8 chips instead of 2, sigh...
Parts:
- renumbered U6 to U2, U7 to U3, U8 to U4, U2 to U5, U3 to U6
Changed lines of the file:
@@
 AR Path="/63A64692" Ref="U?"  Part="1"
 AR Path="/62E48B71/63A64692" Ref="U?"  Part="1"
-AR Path="/63A22C28/63A64692" Ref="U3"  Part="1"
-F 0 "U3" H 10785 4900 50  0000 C CNN
+AR Path="/63A22C28/63A64692" Ref="U6"  Part="1"
+F 0 "U6" H 10785 4900 50  0000 C CNN
 F 1 "74LS257" H 10785 4600 50  0000 C CNN
 F 2 "Package_SO:SOIC-16_3.9x9.9mm_P1.27mm" H 10735 4750 50  0001 C CNN
@@
 AR Path="/63A64698" Ref="U?"  Part="1"
 AR Path="/62E48B71/63A64698" Ref="U?"  Part="1"
-AR Path="/63A22C28/63A64698" Ref="U2"  Part="1"
-F 0 "U2" H 10785 3200 50  0000 C CNN
+AR Path="/63A22C28/63A64698" Ref="U5"  Part="1"
+F 0 "U5" H 10785 3200 50  0000 C CNN
 F 1 "74LS257" H 10785 2900 50  0000 C CNN
 F 2 "Package_SO:SOIC-16_3.9x9.9mm_P1.27mm" H 10735 3050 50  0001 C CNN
@@
 $EndComp
 $Comp
-L 74xx:74LS74 U8
+L 74xx:74LS74 U4
 U 2 1 63CBD2CF
 P 6815 7340
-F 0 "U8" H 6945 7595 50  0000 C CNN
+F 0 "U4" H 6945 7595 50  0000 C CNN
 F 1 "74HCT74" H 6815 7730 50  0001 C CNN
 F 2 "Package_SO:SOIC-14_3.9x8.7mm_P1.27mm" H 6815 7340 50  0001 C CNN
@@
 $EndComp
 $Comp
-L 74xx:74LS74 U7
+L 74xx:74LS74 U3
 U 3 1 63CBF300
 P 1540 10005
-F 0 "U7" H 1770 10051 50  0000 L CNN
+F 0 "U3" H 1770 10051 50  0000 L CNN
 F 1 "74HCT74" H 1770 9960 50  0000 L CNN
 F 2 "Package_SO:SOIC-14_3.9x8.7mm_P1.27mm" H 1540 10005 50  0001 C CNN
@@
 $EndComp
 $Comp
-L 74xx:74LS74 U8
+L 74xx:74LS74 U4
 U 3 1 63CC059A
 P 3105 10005
-F 0 "U8" H 3335 10051 50  0000 L CNN
+F 0 "U4" H 3335 10051 50  0000 L CNN
 F 1 "74HCT74" H 3335 9960 50  0000 L CNN
 F 2 "Package_SO:SOIC-14_3.9x8.7mm_P1.27mm" H 3105 10005 50  0001 C CNN
@@
 Entry Wire Line
 	5420 6080 5520 5980
-$Comp
-L 74xx:74LS74 U8
-U 1 1 63CBBBB2
-P 6285 6795
-F 0 "U8" H 6430 7055 50  0000 C CNN
-F 1 "74HCT74" H 6495 6515 50  0000 C CNN
-F 2 "Package_SO:SOIC-14_3.9x8.7mm_P1.27mm" H 6285 6795 50  0001 C CNN
-F 3 "74xx/74hc_hct74.pdf" H 6285 6795 50  0001 C CNN
-	1    6285 6795
-	1    0    0    -1
-$EndComp
 NoConn ~ 6585 6895
 NoConn ~ 7115 7440
@@
 	5910 7340 6515 7340
 $Comp
-L 74xx:74LS74 U7
+L 74xx:74LS74 U3
 U 2 1 63D2ED5A
 P 6815 6080
-F 0 "U7" H 6945 6335 50  0000 C CNN
+F 0 "U3" H 6945 6335 50  0000 C CNN
 F 1 "74HCT74" H 6815 6470 50  0001 C CNN
 F 2 "Package_SO:SOIC-14_3.9x8.7mm_P1.27mm" H 6815 6080 50  0001 C CNN
@@
 $EndComp
 $Comp
-L 74xx:74LS74 U7
+L 74xx:74LS74 U3
 U 1 1 63D2F89C
 P 6285 5535
-F 0 "U7" H 6430 5795 50  0000 C CNN
+F 0 "U3" H 6430 5795 50  0000 C CNN
 F 1 "74HCT74" H 6495 5255 50  0000 C CNN
 F 2 "Package_SO:SOIC-14_3.9x8.7mm_P1.27mm" H 6285 5535 50  0001 C CNN
@@
 	5090 2960 5190 3060
 $Comp
-L GAL20V8:GAL20V8 U6
+L GAL20V8:GAL20V8 U2
 U 1 1 63F7FBC6
 P 6355 3310
-F 0 "U6" H 6355 4225 50  0000 C CNN
+F 0 "U2" H 6355 4225 50  0000 C CNN
 F 1 "GAL20V8" H 6355 4134 50  0000 C CNN
 F 2 "Package_DIP:DIP-24_W7.62mm_Socket" H 6355 3310 50  0001 C CNN
@@
 Wire Bus Line
 	9285 2250 9285 4950
+$Comp
+L 74xx:74LS74 U4
+U 1 1 63CBBBB2
+P 6285 6795
+F 0 "U4" H 6430 7055 50  0000 C CNN
+F 1 "74HCT74" H 6495 6515 50  0000 C CNN
+F 2 "Package_SO:SOIC-14_3.9x8.7mm_P1.27mm" H 6285 6795 50  0001 C CNN
+F 3 "74xx/74hc_hct74.pdf" H 6285 6795 50  0001 C CNN
+	1    6285 6795
+	1    0    0    -1
+$EndComp
 $EndSCHEMATC

Commit message: Yeah yeah yeah
Parts:
- U5, U6: value 74LS257 -> 74HCT257
Other:
- note added: "'157s WILL BE FINE, TOO"
Changed lines of the file:
@@
 Sheet 3 3
 Title "Hannes256: C16/+4 256 kB RAM Expansion"
-Date "2022-09-19"
+Date "2022-09-26"
 Rev "1git"
 Comp "SukkoPera"
@@
 AR Path="/63A22C28/63A64692" Ref="U6"  Part="1"
 F 0 "U6" H 10785 4900 50  0000 C CNN
-F 1 "74LS257" H 10785 4600 50  0000 C CNN
+F 1 "74HCT257" H 10785 4600 50  0000 C CNN
 F 2 "Package_SO:SOIC-16_3.9x9.9mm_P1.27mm" H 10735 4750 50  0001 C CNN
 F 3 "" H 10735 4750 50  0001 C CNN
@@
 AR Path="/63A22C28/63A64698" Ref="U5"  Part="1"
 F 0 "U5" H 10785 3200 50  0000 C CNN
-F 1 "74LS257" H 10785 2900 50  0000 C CNN
+F 1 "74HCT257" H 10785 2900 50  0000 C CNN
 F 2 "Package_SO:SOIC-16_3.9x9.9mm_P1.27mm" H 10735 3050 50  0001 C CNN
 F 3 "" H 10735 3050 50  0001 C CNN
@@
 	1    0    0    -1
 $EndComp
+Text Notes 10270 3905 0    50   ~ 0
+'157s WILL BE FINE, TOO
 $EndSCHEMATC

Commit message: Add credits
Parts:
- renumbered C7 to C2, C5 to C3, C6 to C4, C1 to C5, C2 to C6
Changed lines of the file:
@@
 Comment1 "Hannes Version (Update 1 with \"TED Feature\")"
 Comment2 "Based on drawings by Solder/Synergy"
-Comment3 ""
+Comment3 "Licensed under CC BY-NC-SA 4.0"
 Comment4 ""
 $EndDescr
@@
 AR Path="/63A64678" Ref="C?"  Part="1"
 AR Path="/62E48B71/63A64678" Ref="C?"  Part="1"
-AR Path="/63A22C28/63A64678" Ref="C7"  Part="1"
-F 0 "C7" H 4530 3256 50  0000 L CNN
+AR Path="/63A22C28/63A64678" Ref="C2"  Part="1"
+F 0 "C2" H 4530 3256 50  0000 L CNN
 F 1 "100n" H 4530 3165 50  0000 L CNN
 F 2 "Capacitor_SMD:C_0805_2012Metric_Pad1.18x1.45mm_HandSolder" H 4453 3060 50  0001 C CNN
@@
 AR Path="/63A6467E" Ref="C?"  Part="1"
 AR Path="/62E48B71/63A6467E" Ref="C?"  Part="1"
-AR Path="/63A22C28/63A6467E" Ref="C2"  Part="1"
-F 0 "C2" H 12600 4701 50  0000 L CNN
+AR Path="/63A22C28/63A6467E" Ref="C6"  Part="1"
+F 0 "C6" H 12600 4701 50  0000 L CNN
 F 1 "100n" H 12600 4610 50  0000 L CNN
 F 2 "Capacitor_SMD:C_0805_2012Metric_Pad1.18x1.45mm_HandSolder" H 12523 4505 50  0001 C CNN
@@
 AR Path="/63A64654" Ref="C?"  Part="1"
 AR Path="/62E48B71/63A64654" Ref="C?"  Part="1"
-AR Path="/63A22C28/63A64654" Ref="C1"  Part="1"
-F 0 "C1" H 12600 3066 50  0000 L CNN
+AR Path="/63A22C28/63A64654" Ref="C5"  Part="1"
+F 0 "C5" H 12600 3066 50  0000 L CNN
 F 1 "100n" H 12600 2975 50  0000 L CNN
 F 2 "Capacitor_SMD:C_0805_2012Metric_Pad1.18x1.45mm_HandSolder" H 12523 2870 50  0001 C CNN
@@
 AR Path="/63ECD15A" Ref="C?"  Part="1"
 AR Path="/62E48B71/63ECD15A" Ref="C?"  Part="1"
-AR Path="/63A22C28/63ECD15A" Ref="C5"  Part="1"
-F 0 "C5" H 915 10051 50  0000 R CNN
+AR Path="/63A22C28/63ECD15A" Ref="C3"  Part="1"
+F 0 "C3" H 915 10051 50  0000 R CNN
 F 1 "100n" H 915 9960 50  0000 R CNN
 F 2 "Capacitor_SMD:C_0805_2012Metric_Pad1.18x1.45mm_HandSolder" H 1068 9855 50  0001 C CNN
@@
 AR Path="/63EDC36A" Ref="C?"  Part="1"
 AR Path="/62E48B71/63EDC36A" Ref="C?"  Part="1"
-AR Path="/63A22C28/63EDC36A" Ref="C6"  Part="1"
-F 0 "C6" H 2480 10051 50  0000 R CNN
+AR Path="/63A22C28/63EDC36A" Ref="C4"  Part="1"
+F 0 "C4" H 2480 10051 50  0000 R CNN
 F 1 "100n" H 2480 9960 50  0000 R CNN
 F 2 "Capacitor_SMD:C_0805_2012Metric_Pad1.18x1.45mm_HandSolder" H 2633 9855 50  0001 C CNN
