File: Hannes256.kicad_pcb (KiCad board)
At the start: 2 copper layers, 56.3 x 82 mm, 38 parts, among them J1 TED_SOCKET, J2 RAM_SELECTOR, J3 CONN_CS, U1 MOS_7360_TED, U10 41256, U11 41256, U12 41256, U13 41256, U14 41256, U15 NE555, U2 GAL20V8, U3 74HCT573, U4 74HCT245, U5 74HCT257, U6 74HCT257, U7 41256, U8 41256, U9 41256

Commit message: Routing in progress
Parts:
- removed C10, C11, C12, C13, C14, C5, C6, C8, C9: 100n, Capacitor_SMD:C_0805_2012Metric_Pad1.18x1.45mm_HandSolder
- removed U10, U11, U12, U13, U14, U7, U8, U9: 41256, Package_DIP:DIP-16_W7.62mm_Socket
- added C1: 100n, Capacitor_SMD:C_0805_2012Metric_Pad1.18x1.45mm_HandSolder, F.Cu at (126.7, 109.0)
- U5: value 74HCT257 -> 74HCT02; footprint Package_SO:SOIC-16_3.9x9.9mm_P1.27mm -> Package_SO:SOIC-14_3.9x8.7mm_P1.27mm
- U6: value 74HCT257 -> AS6C4008; footprint Package_SO:SOIC-16_3.9x9.9mm_P1.27mm -> Package_DIP:DIP-32_W15.24mm_Socket_LongPads
- moved C7 65.0 mm to (148.6, 136.9)
- moved U6 36.2 mm to (156.2, 136.9)
- moved U5 14.6 mm to (126.7, 115.3), turned to 0 degrees
- moved R1 12.1 mm to (132.7, 73.7)
- moved R2 12.1 mm to (120.7, 73.7)
- moved J2 5.08 mm to (129.2, 74.7), turned to 270 degrees
Connections:
- net ~RAS renamed /~ras
- J1 pad 12: /clkout -> CLKOUT
- J1 pad 9: MUX -> /mux
- U1 pad 12: /clkout -> CLKOUT
- U1 pad 9: MUX -> /mux
- U15 pad 4: /~RAS~/~CAS~ Generation/~cs_ramwr -> Net-(U15-Pad4)
- U2 pad 10: MUX -> AEC
- U2 pad 14: p6 -> p2
- U2 pad 15: p7 -> p6
- U2 pad 16: AEC -> p7
- U2 pad 17: Net-(U2-Pad17) -> a18
- U2 pad 18: /~RAS~/~CAS~ Generation/cs_ramwr -> a17
- U2 pad 19: /~RAS~/~CAS~ Generation/~cs_ramrd -> a16
- U2 pad 20: m8 -> /~RAS~/~CAS~ Generation/cs_ramwr
- U2 pad 21: ~CS_OUT -> /~RAS~/~CAS~ Generation/~cs_ramrd
- U2 pad 22: /~RAS~/~CAS~ Generation/~cs_ramwr -> ~CS_OUT
- U5 pad 1: MUX -> ~SRAM_CE
- U5 pad 10: a2 -> Net-(U5-Pad10)
- U5 pad 11: a9 -> /~RAS~/~CAS~ Generation/cs_ramwr
- U5 pad 12: m3 -> /~RAS~/~CAS~ Generation/cs_ramwr
- U5 pad 13: a3 -> Net-(U15-Pad4)
- U5 pad 14: a10 -> +5V
- U5 pad 2: a15 -> Net-(U5-Pad2)
- U5 pad 3: a0 -> Net-(U5-Pad2)
- U5 pad 4: m0 -> Net-(U5-Pad2)
- U5 pad 5: a8 -> Net-(U5-Pad10)
- U5 pad 6: a1 -> ~CAS_64K
- U5 pad 7: m1 -> GND
- U5 pad 8: GND -> CLKOUT
- U5 pad 9: m2 -> R_~W
- U6 pad 1: MUX -> a18
- U6 pad 10: a6 -> a12
- U6 pad 11: a13 -> a14
- U6 pad 12: m7 -> a15
- U6 pad 13: a7 -> d0
- U6 pad 14: a14 -> d1
- U6 pad 15: GND -> d2
- U6 pad 16: +5V -> GND
- U6 pad 2: a11 -> a16
- U6 pad 3: a4 -> a1
- U6 pad 4: m4 -> a0
- U6 pad 5: a12 -> a8
- U6 pad 6: a5 -> a9
- U6 pad 7: m5 -> a10
- U6 pad 8: GND -> a13
- U6 pad 9: m6 -> a11
Routing:
- net m8: track 133.0 -> 0.00 mm
- net m3: track 129.0 -> 0.00 mm, vias 2 -> 0
- net +5V: track 279.7 -> 160.0 mm, vias 11 -> 6
- net m6: track 111.4 -> 0.00 mm, vias 2 -> 0
- net m5: track 103.0 -> 0.00 mm, vias 2 -> 0
- net m2: track 100.9 -> 0.00 mm, vias 1 -> 0
- net m0: track 98.3 -> 0.00 mm
- net m7: track 97.1 -> 0.00 mm
- net m4: track 96.3 -> 0.00 mm
- net m1: track 93.8 -> 0.00 mm
- net /~ras: track 96.0 -> 3.17 mm, vias 1 -> 0
- net R_~W: track 134.0 -> 54.4 mm, vias 1 -> 2
- net a18: track 0.00 -> 78.7 mm, vias 0 -> 1
- net d5: track 133.3 -> 58.4 mm, vias 5 -> 2
- net ~CAS_64K: track 128.5 -> 54.7 mm
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Other:
- board size 56.3 x 82 mm -> 56.3 x 72.2 mm
- board text added: "CC-BY-NC-SA © SukkoPera 2022-2023 github.com/ SukkoPera/ Hannes256"
- board text removed: "CC-BY-NC-SA © SukkoPera 2022 github.com/ SukkoPera/ Hannes256"

Commit message: More routing
Parts:
- moved V0 48.7 mm to (148.3, 120.8), turned to 270 degrees
Connections:
- U6 pad 13: d0 -> d2
- U6 pad 15: d2 -> d0
Routing:
- net d1: track 51.9 -> 83.2 mm, vias 2 -> 4
- net d0: track 60.6 -> 79.4 mm, vias 2 -> 4
- net d2: track 67.7 -> 83.8 mm, vias 2 -> 4
- net d7: track 66.3 -> 78.8 mm
- net d5: track 58.4 -> 68.9 mm, vias 2 -> 3
- net d6: track 82.9 -> 72.5 mm, vias 5 -> 3
- net d3: track 56.6 -> 62.7 mm, vias 2 -> 3
- net +5V: track 160.0 -> 163.9 mm, vias 6 -> 7
- net d4: track 67.1 -> 64.9 mm, vias 4 -> 3
- net a14: track 45.6 -> 47.0 mm
- net a13: track 53.2 -> 52.1 mm
- net a18: track 78.7 -> 79.6 mm
- net Net-(C16-Pad1): track 12.1 -> 11.5 mm
- net ~RESET: track 46.6 -> 47.2 mm
- net /~cas_16k: track 41.9 -> 42.4 mm
Other:
- board text added: "512kB RAM Expansion for the Commodore 16 Based on work by Hannes and Solder/Synergy Thanks to eslapion"
- board text added: "A0"
- board text added: "A1"
- board text added: "A10"
- board text added: "A11"
- board text added: "A12"
- board text added: "A13"
- board text added: "A14"
- board text added: "A15"
- board text added: "A16"
- board text added: "A17"
- board text added: "A18"
- board text added: "A2"
- board text added: "A3"
- board text added: "A4"
- board text added: "A5"
- board text added: "A6"
- board text added: "A7"
- board text added: "A8"
- board text added: "A9"
- board text added: "V4"
- board text removed: "256kB RAM Expansion for the Commodore 16 Based on work by Hannes and Solder/Synergy"
- board text removed: "V2"

Commit message: ROuting done
Parts:
- added V1: LOGO, Hannes256:logo, F.Cu at (140.0, 81.9)
- moved V0 2.95 mm to (148.0, 117.8)
Connections:
- U2 pad 1: a0 -> a1
- U2 pad 11: p0 -> p2
- U2 pad 14: p2 -> p0
- U2 pad 2: a1 -> a2
- U2 pad 3: a2 -> a3
- U2 pad 4: a3 -> a0
Routing:
- net +5V: track 163.9 -> 237.2 mm, vias 7 -> 10
- net /~RAS~/~CAS~ Generation/cs_ramwr: track 11.7 -> 53.0 mm, vias 1 -> 2
- net /~RAS~/~CAS~ Generation/~cs_ramrd: track 25.7 -> 57.7 mm, vias 1 -> 2
- net a0: track 24.5 -> 56.3 mm
- net a2: track 33.4 -> 63.7 mm, vias 0 -> 1
- net p2: track 17.9 -> 35.1 mm, vias 2 -> 3
- net a1: track 52.0 -> 49.2 mm
- net ~CS_IN: track 18.3 -> 19.7 mm
- net p1: track 34.5 -> 33.2 mm
- net a11: track 42.6 -> 41.4 mm
- net p0: track 32.9 -> 34.0 mm
- net Net-(U15-Pad4): track 14.8 -> 13.8 mm
- net a16: track 71.5 -> 72.4 mm
- net ~RESET: track 47.2 -> 48.1 mm
- net a13: track 52.1 -> 51.4 mm
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Other:
- board size 56.3 x 72.2 mm -> 54.3 x 72.2 mm
- board text added: "512K"
- board text added: "512kB RAM Expansion for the Commodore 16 Based on work by Hannes and Solder/Synergy Thanks to TLC and eslapion"
- board text added: "D0"
- board text added: "D1"
- board text added: "D2"
- board text added: "D3"
- board text added: "D4"
- board text added: "D5"
- board text added: "D6"
- board text added: "D7"
- board text removed: "256K"
- board text removed: "512kB RAM Expansion for the Commodore 16 Based on work by Hannes and Solder/Synergy Thanks to eslapion"

Commit message: Relabel all components
Parts:
- moved C5 3.81 mm to (110.1, 83.6)
- moved C6 3.81 mm to (110.1, 79.8)
- renumbered C7 to C1, C1 to C2, C16 to C3, C15 to C4, C3 to C5, C4 to C6, C2 to C7, J1 to J0, J3 to J1, U6 to U2, U5 to U3, U15 to U4, U3 to U5, U4 to U6, U2 to U7, V0 to V1, V1 to V2
